File: 03_usb_adapter.kicad_sch (KiCad schematic)
At the start: 24 parts, among them J1 Conn_02x05_Odd_Even, J2 Conn_01x04_Male, J3 Conn_01x02_Male, U2 CYUSB306X, U4 ECS-1612MV-192-CN-TR, U5 74LVC2G17

Commit message: finished schematics
Parts:
- C33, C34: footprint (none) -> Capacitor_SMD:C_0603_1608Metric
- J3: footprint (none) -> Connector_PinSocket_2.00mm:PinSocket_1x02_P2.00mm_Vertical
Connections:
- net +3.3V is gone; now on net +3V3: R16.1, R18.1
- net VCC is gone; now on net +3V3: U5.5 (VCC), U5.5 (VCC)
- no-connect marks 27 -> 28
Other:
- moved on the sheet: U5A
Changed lines of the file:
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@@
   (junction (at 46.99 121.92) (diameter 0) (color 0 0 0 0)
   )
+  (junction (at 99.06 168.91) (diameter 0) (color 0 0 0 0)
+  )
   (junction (at 200.66 50.8) (diameter 0) (color 0 0 0 0)
-  )
-  (junction (at 99.06 168.91) (diameter 0) (color 0 0 0 0)
   )
   (junction (at 196.85 151.13) (diameter 0) (color 0 0 0 0)
@@
   (no_connect (at 254 74.93))
   (no_connect (at 254 90.17))
+  (no_connect (at 213.36 90.17))
   (no_connect (at 254 49.53))
   (no_connect (at 254 72.39))
@@
     (stroke (width 0) (type default) (color 0 0 0 0))
   )
-  (wire (pts (xy 99.06 168.91) (xy 106.68 168.91))
-    (stroke (width 0) (type default) (color 0 0 0 0))
-  )
   (wire (pts (xy 55.88 93.98) (xy 67.31 93.98))
     (stroke (width 0) (type default) (color 0 0 0 0))
   )
+  (wire (pts (xy 99.06 156.21) (xy 99.06 168.91))
+    (stroke (width 0) (type default) (color 0 0 0 0))
+  )
   (wire (pts (xy 212.09 151.13) (xy 215.9 151.13))
     (stroke (width 0) (type default) (color 0 0 0 0))
@@
     (stroke (width 0) (type default) (color 0 0 0 0))
   )
+  (wire (pts (xy 106.68 156.21) (xy 99.06 156.21))
+    (stroke (width 0) (type default) (color 0 0 0 0))
+  )
   (wire (pts (xy 53.34 161.29) (xy 53.34 162.56))
     (stroke (width 0) (type default) (color 0 0 0 0))
@@
     (stroke (width 0) (type default) (color 0 0 0 0))
   )
+  (wire (pts (xy 114.3 177.8) (xy 114.3 180.34))
+    (stroke (width 0) (type default) (color 0 0 0 0))
+  )
   (wire (pts (xy 64.77 119.38) (xy 71.12 119.38))
     (stroke (width 0) (type default) (color 0 0 0 0))
@@
     (stroke (width 0) (type default) (color 0 0 0 0))
   )
-  (wire (pts (xy 120.65 168.91) (xy 138.43 168.91))
+  (wire (pts (xy 120.65 156.21) (xy 138.43 156.21))
     (stroke (width 0) (type default) (color 0 0 0 0))
   )
@@
     (stroke (width 0) (type default) (color 0 0 0 0))
   )
+  (wire (pts (xy 114.3 158.75) (xy 114.3 161.29))
+    (stroke (width 0) (type default) (color 0 0 0 0))
+  )
   (wire (pts (xy 106.68 182.88) (xy 99.06 182.88))
     (stroke (width 0) (type default) (color 0 0 0 0))
@@
   )
   (wire (pts (xy 72.39 168.91) (xy 63.5 168.91))
+    (stroke (width 0) (type default) (color 0 0 0 0))
+  )
+  (wire (pts (xy 114.3 185.42) (xy 114.3 187.96))
+    (stroke (width 0) (type default) (color 0 0 0 0))
+  )
+  (wire (pts (xy 114.3 149.86) (xy 114.3 153.67))
     (stroke (width 0) (type default) (color 0 0 0 0))
   )
@@
     (effects (font (size 1.27 1.27)) (justify left bottom))
   )
-  (label "OSC_19M2" (at 138.43 168.91 180)
+  (label "OSC_19M2" (at 138.43 156.21 180)
     (effects (font (size 1.27 1.27)) (justify right bottom))
   )
@@
     (property "Reference" "J3" (id 0) (at 180.975 87.63 0))
     (property "Value" "Conn_01x02_Male" (id 1) (at 180.975 90.17 0))
-    (property "Footprint" "" (id 2) (at 180.34 92.71 0)
+    (property "Footprint" "Connector_PinSocket_2.00mm:PinSocket_1x02_P2.00mm_Vertical" (id 2) (at 180.34 92.71 0)
       (effects (font (size 1.27 1.27)) hide)
     )
@@
     (pin "1")
     (pin "2")
+  )
+  (symbol (lib_id "power:+3V3") (at 190.5 80.01 0) (unit 1)
+    (in_bom yes) (on_board yes)
+    (property "Reference" "#PWR0121" (id 0) (at 190.5 83.82 0)
+      (effects (font (size 1.27 1.27)) hide)
+    )
+    (property "Value" "+3V3" (id 1) (at 190.881 75.6158 0))
+    (property "Footprint" "" (id 2) (at 190.5 80.01 0)
+      (effects (font (size 1.27 1.27)) hide)
+    )
+    (property "Datasheet" "" (id 3) (at 190.5 80.01 0)
+      (effects (font (size 1.27 1.27)) hide)
+    )
+    (pin "1")
   )
   (symbol (lib_id "Device:R") (at 200.66 45.72 0) (unit 1)
@@
     (property "Reference" "C33" (id 0) (at 57.15 41.91 90))
     (property "Value" "100n" (id 1) (at 66.04 41.91 90))
-    (property "Footprint" "" (id 2) (at 64.77 42.2148 0)
+    (property "Footprint" "Capacitor_SMD:C_0603_1608Metric" (id 2) (at 64.77 42.2148 0)
       (effects (font (size 1.27 1.27)) hide)
     )
@@
     (pin "2")
   )
-  (symbol (lib_id "power:+3.3V") (at 199.39 80.01 0) (unit 1)
-    (in_bom yes) (on_board yes) (fields_autoplaced)
-    (property "Reference" "#PWR076" (id 0) (at 199.39 83.82 0)
-      (effects (font (size 1.27 1.27)) hide)
-    )
-    (property "Value" "+3.3V" (id 1) (at 199.39 74.93 0))
-    (property "Footprint" "" (id 2) (at 199.39 80.01 0)
-      (effects (font (size 1.27 1.27)) hide)
-    )
-    (property "Datasheet" "" (id 3) (at 199.39 80.01 0)
+  (symbol (lib_id "power:GND") (at 114.3 161.29 0) (unit 1)
+    (in_bom yes) (on_board yes) (fields_autoplaced)
+    (property "Reference" "#PWR0117" (id 0) (at 114.3 167.64 0)
+      (effects (font (size 1.27 1.27)) hide)
+    )
+    (property "Value" "GND" (id 1) (at 114.3 166.37 0))
+    (property "Footprint" "" (id 2) (at 114.3 161.29 0)
+      (effects (font (size 1.27 1.27)) hide)
+    )
+    (property "Datasheet" "" (id 3) (at 114.3 161.29 0)
       (effects (font (size 1.27 1.27)) hide)
     )
@@
     (property "Reference" "C34" (id 0) (at 68.58 39.37 90))
     (property "Value" "100n" (id 1) (at 76.2 39.37 90))
-    (property "Footprint" "" (id 2) (at 76.2 39.6748 0)
+    (property "Footprint" "Capacitor_SMD:C_0603_1608Metric" (id 2) (at 76.2 39.6748 0)
       (effects (font (size 1.27 1.27)) hide)
     )
@@
   )
   (symbol (lib_id "74xGxx:74LVC2G17") (at 114.3 182.88 0) (unit 2)
-    (in_bom yes) (on_board yes) (fields_autoplaced)
-    (property "Reference" "U5" (id 0) (at 113.665 175.26 0))
-    (property "Value" "74LVC2G17" (id 1) (at 113.665 177.8 0))
+    (in_bom yes) (on_board yes)
+    (property "Reference" "U5" (id 0) (at 118.11 176.53 0))
+    (property "Value" "74LVC2G17" (id 1) (at 121.92 179.07 0))
     (property "Footprint" "Package_TO_SOT_SMD:SOT-363_SC-70-6" (id 2) (at 114.3 182.88 0)
       (effects (font (size 1.27 1.27)) hide)
@@
     (pin "3")
     (pin "4")
+  )
+  (symbol (lib_id "power:+3V3") (at 114.3 177.8 0) (unit 1)
+    (in_bom yes) (on_board yes) (fields_autoplaced)
+    (property "Reference" "#PWR0116" (id 0) (at 114.3 181.61 0)
+      (effects (font (size 1.27 1.27)) hide)
+    )
+    (property "Value" "+3V3" (id 1) (at 114.3 172.72 0))
+    (property "Footprint" "" (id 2) (at 114.3 177.8 0)
+      (effects (font (size 1.27 1.27)) hide)
+    )
+    (property "Datasheet" "" (id 3) (at 114.3 177.8 0)
+      (effects (font (size 1.27 1.27)) hide)
+    )
+    (pin "1")
   )
   (symbol (lib_id "Connector_Generic:Conn_02x05_Odd_Even") (at 57.15 121.92 0) (unit 1)
@@
     (pin "2")
   )
-  (symbol (lib_id "power:+3.3V") (at 190.5 80.01 0) (unit 1)
-    (in_bom yes) (on_board yes) (fields_autoplaced)
-    (property "Reference" "#PWR074" (id 0) (at 190.5 83.82 0)
-      (effects (font (size 1.27 1.27)) hide)
-    )
-    (property "Value" "+3.3V" (id 1) (at 190.5 74.93 0))
-    (property "Footprint" "" (id 2) (at 190.5 80.01 0)
-      (effects (font (size 1.27 1.27)) hide)
-    )
-    (property "Datasheet" "" (id 3) (at 190.5 80.01 0)
+  (symbol (lib_id "power:GND") (at 114.3 187.96 0) (unit 1)
+    (in_bom yes) (on_board yes) (fields_autoplaced)
+    (property "Reference" "#PWR0115" (id 0) (at 114.3 194.31 0)
+      (effects (font (size 1.27 1.27)) hide)
+    )
+    (property "Value" "GND" (id 1) (at 114.3 193.04 0))
+    (property "Footprint" "" (id 2) (at 114.3 187.96 0)
+      (effects (font (size 1.27 1.27)) hide)
+    )
+    (property "Datasheet" "" (id 3) (at 114.3 187.96 0)
       (effects (font (size 1.27 1.27)) hide)
     )
@@
     (pin "1")
     (pin "2")
+  )
+  (symbol (lib_id "power:+3V3") (at 114.3 149.86 0) (unit 1)
+    (in_bom yes) (on_board yes) (fields_autoplaced)
+    (property "Reference" "#PWR0118" (id 0) (at 114.3 153.67 0)
+      (effects (font (size 1.27 1.27)) hide)
+    )
+    (property "Value" "+3V3" (id 1) (at 114.3 144.78 0))
+    (property "Footprint" "" (id 2) (at 114.3 149.86 0)
+      (effects (font (size 1.27 1.27)) hide)
+    )
+    (property "Datasheet" "" (id 3) (at 114.3 149.86 0)
+      (effects (font (size 1.27 1.27)) hide)
+    )
+    (pin "1")
   )
   (symbol (lib_id "Device:R") (at 199.39 86.36 0) (unit 1)
@@
     (pin "F6")
   )
+  (symbol (lib_id "power:+3V3") (at 199.39 80.01 0) (unit 1)
+    (in_bom yes) (on_board yes)
+    (property "Reference" "#PWR0120" (id 0) (at 199.39 83.82 0)
+      (effects (font (size 1.27 1.27)) hide)
+    )
+    (property "Value" "+3V3" (id 1) (at 199.771 75.6158 0))
+    (property "Footprint" "" (id 2) (at 199.39 80.01 0)
+      (effects (font (size 1.27 1.27)) hide)
+    )
+    (property "Datasheet" "" (id 3) (at 199.39 80.01 0)
+      (effects (font (size 1.27 1.27)) hide)
+    )
+    (pin "1")
+  )
   (symbol (lib_id "Device:R") (at 74.93 124.46 90) (unit 1)
     (in_bom yes) (on_board yes)
@@
     (pin "1")
   )
-  (symbol (lib_id "74xGxx:74LVC2G17") (at 114.3 168.91 0) (unit 1)
-    (in_bom yes) (on_board yes) (fields_autoplaced)
-    (property "Reference" "U5" (id 0) (at 113.665 161.29 0))
-    (property "Value" "74LVC2G17" (id 1) (at 113.665 163.83 0))
-    (property "Footprint" "Package_TO_SOT_SMD:SOT-363_SC-70-6" (id 2) (at 114.3 168.91 0)
-      (effects (font (size 1.27 1.27)) hide)
-    )
-    (property "Datasheet" "http://www.ti.com/lit/sg/scyt129e/scyt129e.pdf" (id 3) (at 114.3 168.91 0)
-      (effects (font (size 1.27 1.27)) hide)
-    )
+  (symbol (lib_id "74xGxx:74LVC2G17") (at 114.3 156.21 0) (unit 1)
+    (in_bom yes) (on_board yes)
+    (property "Reference" "U5" (id 0) (at 119.38 148.59 0))
+    (property "Value" "74LVC2G17" (id 1) (at 121.92 151.13 0))
+    (property "Footprint" "Package_TO_SOT_SMD:SOT-363_SC-70-6" (id 2) (at 114.3 156.21 0)
+      (effects (font (size 1.27 1.27)) hide)
+    )
+    (property "Datasheet" "http://www.ti.com/lit/sg/scyt129e/scyt129e.pdf" (id 3) (at 114.3 156.21 0)
+      (effects (font (size 1.27 1.27)) hide)
+    )
